File: Dot_LED_Matrix_driver_board.sch (KiCad schematic (older format))
At the start: 9 parts, among them U1 MAX7219

Commit message: Signed-off-by: Martynas Sprogys <msp@dancerbus.com>
Parts:
- C1: footprint (none) -> Capacitor_SMD:C_1206_3216Metric_Pad1.42x1.75mm_HandSolder
- C2: footprint (none) -> Capacitor_SMD:CP_Elec_5x3
- DATA_IN1, DATA_OUT1: footprint (none) -> Connector_PinHeader_1.27mm:PinHeader_1x05_P1.27mm_Vertical
- R1, R2: footprint (none) -> Resistor_SMD:R_1206_3216Metric_Pad1.42x1.75mm_HandSolder
Changed lines of the file:
@@
 F 0 "R2" H 6870 3896 50  0000 L CNN
 F 1 "27k" H 6870 3805 50  0000 L CNN
-F 2 "" V 6730 3850 50  0001 C CNN
+F 2 "Resistor_SMD:R_1206_3216Metric_Pad1.42x1.75mm_HandSolder" V 6730 3850 50  0001 C CNN
 F 3 "~" H 6800 3850 50  0001 C CNN
 	1    6800 3850
@@
 F 0 "C1" H 6015 3896 50  0000 L CNN
 F 1 "0,1uF" H 6015 3805 50  0000 L CNN
-F 2 "" H 5938 3700 50  0001 C CNN
+F 2 "Capacitor_SMD:C_1206_3216Metric_Pad1.42x1.75mm_HandSolder" H 5938 3700 50  0001 C CNN
 F 3 "~" H 5900 3850 50  0001 C CNN
 	1    5900 3850
@@
 F 0 "C2" H 6515 3896 50  0000 L CNN
 F 1 "10uF" H 6515 3805 50  0000 L CNN
-F 2 "" H 6400 3850 50  0001 C CNN
+F 2 "Capacitor_SMD:CP_Elec_5x3" H 6400 3850 50  0001 C CNN
 F 3 "~" H 6400 3850 50  0001 C CNN
 	1    6400 3850
@@
 F 0 "DATA_IN1" H 4020 6292 50  0000 L CNN
 F 1 "Conn_01x05" H 4020 6201 50  0000 L CNN
-F 2 "" H 3940 6250 50  0001 C CNN
+F 2 "Connector_PinHeader_1.27mm:PinHeader_1x05_P1.27mm_Vertical" H 3940 6250 50  0001 C CNN
 F 3 "~" H 3940 6250 50  0001 C CNN
 	1    3940 6250
@@
 F 0 "DATA_OUT1" H 4030 7292 50  0000 L CNN
 F 1 "Conn_01x05" H 4030 7201 50  0000 L CNN
-F 2 "" H 3950 7250 50  0001 C CNN
+F 2 "Connector_PinHeader_1.27mm:PinHeader_1x05_P1.27mm_Vertical" H 3950 7250 50  0001 C CNN
 F 3 "~" H 3950 7250 50  0001 C CNN
 	1    3950 7250
@@
 F 0 "R1" H 6540 5696 50  0000 L CNN
 F 1 "10k" H 6540 5605 50  0000 L CNN
-F 2 "" V 6400 5650 50  0001 C CNN
+F 2 "Resistor_SMD:R_1206_3216Metric_Pad1.42x1.75mm_HandSolder" V 6400 5650 50  0001 C CNN
 F 3 "~" H 6470 5650 50  0001 C CNN
 	1    6470 5650

Commit message: Update
Signed-off-by: Martynas Sprogys <martynas2580@gmail.com>
Changed lines of the file:
@@
 	6800 4100 6900 4100
-Wire Wire Line
-	7300 3890 7300 3670
 Wire Wire Line
 	6800 3700 6800 3670
 Wire Wire Line
 	6800 3670 7300 3670
-Connection ~ 7300 3670
 Wire Wire Line
 	7300 3670 7300 3610
@@
 	1    0    0    -1
 $EndComp
-Connection ~ 6470 5500
 $Comp
 L power:GND #PWR0104
@@
 Wire Wire Line
 	6470 5900 6470 5800
-Wire Wire Line
-	6470 5500 6890 5500
 Text GLabel 6900 5600 0    50   Input ~ 0
 CK
@@
 Text GLabel 3750 7250 0    50   Input ~ 0
 DOUT
+Wire Wire Line
+	7300 3900 7300 3670
+Connection ~ 7300 3670
+Wire Wire Line
+	6470 5500 6900 5500
+Connection ~ 6470 5500
 $EndSCHEMATC
