File: Dot_LED_Matrix_driver_board.kicad_pcb (KiCad board)
At the start: 2 copper layers, 3 parts, among them J1 Conn_01x08, J2 Conn_01x08, U1 MAX7219

Commit message: Signed-off-by: Martynas Sprogys <msp@dancerbus.com>
Parts:
- removed J1: Conn_01x08, Connector_PinHeader_2.54mm:PinHeader_1x08_P2.54mm_Vertical
- added Anodes(+)1: pin header 2.54 mm, Connector_PinHeader_2.54mm:PinHeader_1x08_P2.54mm_Vertical, F.Cu at (121.2, 77.2)
- added C1: 0,1uF, Capacitor_SMD:C_1206_3216Metric_Pad1.42x1.75mm_HandSolder, F.Cu at (227.5, 65.0)
- added C2: 10uF, Capacitor_SMD:CP_Elec_5x3, F.Cu at (220.1, 66.8)
- added DATA_IN1: Conn_01x05, Connector_PinHeader_1.27mm:PinHeader_1x05_P1.27mm_Vertical, F.Cu at (223.5, 90.5)
- added DATA_OUT1: Conn_01x05, Connector_PinHeader_1.27mm:PinHeader_1x05_P1.27mm_Vertical, F.Cu at (223.5, 81.5)
- added R1: 10k, Resistor_SMD:R_1206_3216Metric_Pad1.42x1.75mm_HandSolder, F.Cu at (227.5, 68.3)
- added R2: 27k, Resistor_SMD:R_1206_3216Metric_Pad1.42x1.75mm_HandSolder, F.Cu at (227.5, 71.6)
- Cathodes(-)1: renamed from J2; value Conn_01x08 -> pin header 2.54 mm
- moved Cathodes(-)1 24.6 mm to (121.2, 123.0)
- moved U1 16.9 mm to (128.7, 99.2)
Connections:
- net Net-(U1-Pad4) renamed GND
- Cathodes(-)1 pad 1: Net-(J2-Pad1) -> 9
- Cathodes(-)1 pad 2: Net-(J2-Pad2) -> 10
- Cathodes(-)1 pad 3: Net-(J2-Pad3) -> 11
- Cathodes(-)1 pad 4: Net-(J2-Pad4) -> 12
- Cathodes(-)1 pad 5: Net-(J2-Pad5) -> 13
- Cathodes(-)1 pad 6: Net-(J2-Pad6) -> 14
- Cathodes(-)1 pad 7: Net-(J2-Pad7) -> 15
- Cathodes(-)1 pad 8: Net-(J2-Pad8) -> 16
- U1 pad 1: Net-(U1-Pad1) -> DIN
- U1 pad 10: Net-(U1-Pad10) -> 7
- U1 pad 11: Net-(U1-Pad11) -> 14
- U1 pad 13: Net-(U1-Pad13) -> CK
- U1 pad 14: Net-(U1-Pad14) -> 3
- U1 pad 15: Net-(U1-Pad15) -> 15
- U1 pad 16: Net-(U1-Pad16) -> 4
- U1 pad 17: Net-(U1-Pad17) -> 16
- U1 pad 2: Net-(U1-Pad2) -> 9
- U1 pad 20: Net-(U1-Pad20) -> 10
- U1 pad 21: Net-(U1-Pad21) -> 11
- U1 pad 22: Net-(U1-Pad22) -> 13
- U1 pad 23: Net-(U1-Pad23) -> 6
- U1 pad 24: Net-(U1-Pad24) -> DOUT
- U1 pad 3: Net-(U1-Pad3) -> 1
- U1 pad 5: Net-(U1-Pad5) -> 2
- U1 pad 6: Net-(U1-Pad6) -> 8
- U1 pad 7: Net-(U1-Pad7) -> 12
- U1 pad 8: Net-(U1-Pad8) -> 5

Commit message: second commit
Signed-off-by: Martynas Sprogys <martynas2580@gmail.com>
Parts:
- Anodes(+)1, Cathodes(-)1: moved to B.Cu
- U1: moved to F.Cu
- turned Anodes(+)1 to 270 degrees
- turned Cathodes(-)1 to 270 degrees

Commit message: Update
Signed-off-by: Martynas Sprogys <martynas2580@gmail.com>
Parts:
- moved DATA_IN1 119.1 mm to (105.0, 102.6), turned to 180 degrees
- moved R2 111.2 mm to (125.6, 116.2), turned to 180 degrees
- moved C1 107.4 mm to (129.0, 107.8), turned to 180 degrees
- moved R1 106.6 mm to (123.1, 90.0), turned to 90 degrees
- moved C2 103.1 mm to (127.5, 112.1), turned to 180 degrees
- moved DATA_OUT1 71.7 mm to (155.0, 102.6), turned to 180 degrees
- moved Cathodes(-)1 17.8 mm to (139.0, 123.0), turned to 90 degrees
- moved U1 1.66 mm to (130.1, 100.1), turned to 270 degrees
Connections:
- U1 pad 12: Net-(U1-Pad12) -> CS
- U1 pad 19: Net-(U1-Pad19) -> 5V
Routing:
- net CK: track 0.00 -> 94.2 mm, vias 0 -> 2
- net 5V: track 0.00 -> 65.1 mm
- net CS: track 0.00 -> 57.4 mm
- net 1: track 0.00 -> 45.4 mm
- net 14: track 0.00 -> 42.7 mm, vias 0 -> 2
- net DIN: track 0.00 -> 40.0 mm, vias 0 -> 2
- net 3: track 0.00 -> 29.1 mm, vias 0 -> 2
- net 9: track 0.00 -> 28.6 mm, vias 0 -> 2
- net 4: track 0.00 -> 28.3 mm, vias 0 -> 2
- net 12: track 0.00 -> 28.3 mm, vias 0 -> 2
- net 6: track 0.00 -> 28.3 mm, vias 0 -> 1
- net 16: track 0.00 -> 25.2 mm, vias 0 -> 2
- net 2: track 0.00 -> 25.0 mm, vias 0 -> 2
- net 7: track 0.00 -> 24.9 mm, vias 0 -> 2
- net DOUT: track 0.00 -> 24.6 mm
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- added copper zone on B.Cu, net GND
- added copper zone on F.Cu, net GND
Other:
- board outline added: 60.2 x 60.2 mm
- board text added: "."
- board text added: "0,1 uF"
- board text added: "1"
- board text added: "10k"
- board text added: "10uF"
- board text added: "16"
- board text added: "27k"
- board text added: "8"
- board text added: "9"
- board text added: "MAX7219"

Commit message: Update 01/13
Signed-off-by: Martynas Sprogys <martynas2580@gmail.com>
Other:
- board text added: "Note: 1)5V 2)GND 3)DOUT 4)SCK (LOAD) 5)CLOCK"
- board text added: "Note: 1)5V 2)GND 3)MOSI (DIN) 4)SCK (LOAD) 5)CLOCK"

Commit message: Include silk data on the board
Signed-off-by: Martynas Sprogys <martynas2580@gmail.com>
Other:
- net class Default removed

Commit message: Push
Signed-off-by: Martynas Sprogys <martynas2580@gmail.com>
Other:
- board text added: "v.1"
Changed lines of the file:
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@@
     (effects (font (size 1 1) (thickness 0.15)) (justify left))
+  )
+  (gr_text "v.1" (at 155.3 127.4) (layer "F.SilkS")
+    (effects (font (size 1 1) (thickness 0.2)))
   )
   (gr_text "." (at 137.1 93.1) (layer "F.SilkS")

Commit message: Signed-off-by: Martynas Sprogys <martynas2580@gmail.com>
Parts:
- removed the Anodes(+)1 at (121.2, 77.2)
- removed the C1 at (129.0, 107.8)
- removed the C2 at (127.5, 112.1)
- removed the Cathodes(-)1 at (139.0, 123.0)
- removed the DATA_IN1 at (105.0, 102.6)
- removed the DATA_OUT1 at (155.0, 102.6)
- removed the R1 at (123.1, 90.0)
- removed the R2 at (125.6, 116.2)
- removed the U1 at (130.1, 100.1)
- added Anodes(+)1: pin header 2.54 mm, Connector_PinHeader_2.54mm:PinHeader_1x08_P2.54mm_Vertical, B.Cu at (41.1, 92.3)
- added Anodes(+)1: pin header 2.54 mm, Connector_PinHeader_2.54mm:PinHeader_1x08_P2.54mm_Vertical, B.Cu at (41.1, 27.1)
- added Anodes(+)1: pin header 2.54 mm, Connector_PinHeader_2.54mm:PinHeader_1x08_P2.54mm_Vertical, B.Cu at (106.3, 27.1)
- added Anodes(+)1: pin header 2.54 mm, Connector_PinHeader_2.54mm:PinHeader_1x08_P2.54mm_Vertical, B.Cu at (124.1, 138.1)
- added C1: 0,1uF, Capacitor_SMD:C_1206_3216Metric_Pad1.42x1.75mm_HandSolder, F.Cu at (116.3, 107.5)
- added C1: 0,1uF, Capacitor_SMD:C_1206_3216Metric_Pad1.42x1.75mm_HandSolder, F.Cu at (48.9, 57.7)
- added C1: 0,1uF, Capacitor_SMD:C_1206_3216Metric_Pad1.42x1.75mm_HandSolder, F.Cu at (114.1, 57.7)
- added C1: 0,1uF, Capacitor_SMD:C_1206_3216Metric_Pad1.42x1.75mm_HandSolder, F.Cu at (48.9, 122.9)
- added C2: 10uF, Capacitor_SMD:CP_Elec_5x3, F.Cu at (47.4, 62.0)
- added C2: 10uF, Capacitor_SMD:CP_Elec_5x3, F.Cu at (117.8, 103.2)
- added C2: 10uF, Capacitor_SMD:CP_Elec_5x3, F.Cu at (47.4, 127.2)
- added C2: 10uF, Capacitor_SMD:CP_Elec_5x3, F.Cu at (112.6, 62.0)
- added Cathodes(-)1: pin header 2.54 mm, Connector_PinHeader_2.54mm:PinHeader_1x08_P2.54mm_Vertical, B.Cu at (58.9, 72.9)
- added Cathodes(-)1: pin header 2.54 mm, Connector_PinHeader_2.54mm:PinHeader_1x08_P2.54mm_Vertical, B.Cu at (58.9, 138.1)
- added Cathodes(-)1: pin header 2.54 mm, Connector_PinHeader_2.54mm:PinHeader_1x08_P2.54mm_Vertical, B.Cu at (106.3, 92.3)
- added Cathodes(-)1: pin header 2.54 mm, Connector_PinHeader_2.54mm:PinHeader_1x08_P2.54mm_Vertical, B.Cu at (124.1, 72.9)
- added DATA_IN1: Conn_01x05, Connector_PinHeader_1.27mm:PinHeader_1x05_P1.27mm_Vertical, F.Cu at (24.9, 117.7)
- added DATA_IN1: Conn_01x05, Connector_PinHeader_1.27mm:PinHeader_1x05_P1.27mm_Vertical, F.Cu at (24.9, 52.5)
- added DATA_IN1: Conn_01x05, Connector_PinHeader_1.27mm:PinHeader_1x05_P1.27mm_Vertical, F.Cu at (90.1, 52.5)
- added DATA_IN1: Conn_01x05, Connector_PinHeader_1.27mm:PinHeader_1x05_P1.27mm_Vertical, F.Cu at (140.3, 112.7)
- added DATA_OUT1: Conn_01x05, Connector_PinHeader_1.27mm:PinHeader_1x05_P1.27mm_Vertical, F.Cu at (90.3, 112.7)
- added DATA_OUT1: Conn_01x05, Connector_PinHeader_1.27mm:PinHeader_1x05_P1.27mm_Vertical, F.Cu at (140.1, 52.5)
- added DATA_OUT1: Conn_01x05, Connector_PinHeader_1.27mm:PinHeader_1x05_P1.27mm_Vertical, F.Cu at (74.9, 117.7)
- added DATA_OUT1: Conn_01x05, Connector_PinHeader_1.27mm:PinHeader_1x05_P1.27mm_Vertical, F.Cu at (74.9, 52.5)
- added R1: 10k, Resistor_SMD:R_1206_3216Metric_Pad1.42x1.75mm_HandSolder, F.Cu at (108.2, 39.9)
- added R1: 10k, Resistor_SMD:R_1206_3216Metric_Pad1.42x1.75mm_HandSolder, F.Cu at (122.2, 125.3)
- added R1: 10k, Resistor_SMD:R_1206_3216Metric_Pad1.42x1.75mm_HandSolder, F.Cu at (43.0, 39.9)
- added R1: 10k, Resistor_SMD:R_1206_3216Metric_Pad1.42x1.75mm_HandSolder, F.Cu at (43.0, 105.1)
- added R2: 27k, Resistor_SMD:R_1206_3216Metric_Pad1.42x1.75mm_HandSolder, F.Cu at (45.5, 66.1)
- added R2: 27k, Resistor_SMD:R_1206_3216Metric_Pad1.42x1.75mm_HandSolder, F.Cu at (45.5, 131.3)
- added R2: 27k, Resistor_SMD:R_1206_3216Metric_Pad1.42x1.75mm_HandSolder, F.Cu at (110.7, 66.1)
- added R2: 27k, Resistor_SMD:R_1206_3216Metric_Pad1.42x1.75mm_HandSolder, F.Cu at (119.7, 99.1)
- added U1: MAX7219, Package_SO:SOP-24_7.5x15.4mm_P1.27mm, F.Cu at (50.0, 115.2)
- added U1: MAX7219, Package_SO:SOP-24_7.5x15.4mm_P1.27mm, F.Cu at (50.0, 50.0)
- added U1: MAX7219, Package_SO:SOP-24_7.5x15.4mm_P1.27mm, F.Cu at (115.2, 50.0)
- added U1: MAX7219, Package_SO:SOP-24_7.5x15.4mm_P1.27mm, F.Cu at (115.2, 115.2)
Routing:
- net Board_1-CK: track 0.00 -> 94.2 mm, vias 0 -> 2
- net Board_2-CK: track 0.00 -> 94.2 mm, vias 0 -> 2
- net Board_0-CK: track 0.00 -> 94.2 mm, vias 0 -> 2
- net CK: track 94.2 -> 0.00 mm, vias 2 -> 0
- net Board_3-CK: track 0.00 -> 94.2 mm, vias 0 -> 2
- net 5V: track 65.1 -> 0.00 mm
- net Board_3-5V: track 0.00 -> 65.1 mm
- net Board_2-5V: track 0.00 -> 65.1 mm
- net Board_1-5V: track 0.00 -> 65.1 mm
- net Board_0-5V: track 0.00 -> 65.1 mm
- net CS: track 57.4 -> 0.00 mm
- net Board_3-CS: track 0.00 -> 57.4 mm
- net Board_2-CS: track 0.00 -> 57.4 mm
- net Board_0-CS: track 0.00 -> 57.4 mm
- net Board_1-CS: track 0.00 -> 57.4 mm
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- added copper zone on B.Cu, net Board_0-GND
- added copper zone on F.Cu, net Board_0-GND
- added copper zone on B.Cu, net Board_1-GND
- added copper zone on F.Cu, net Board_1-GND
- added copper zone on B.Cu, net Board_2-GND
- added copper zone on F.Cu, net Board_2-GND
- added copper zone on B.Cu, net Board_3-GND
- added copper zone on F.Cu, net Board_3-GND
- removed copper zone on B.Cu, net GND
- removed copper zone on F.Cu, net GND
Other:
- board size 60.2 x 60.2 mm -> 125.4 x 125.4 mm
